File: comma_connector.kicad_pcb (KiCad board)
At the start: 2 copper layers, 37 x 59.5 mm, 2 parts, among them J1 2317507-1, J2 Screw_Terminal_01x12

Commit message: minor updates to PCB
Parts:
- moved J1 1.00 mm to (201.5, 103.0)
Routing:
- net Net-(J2-Pin_9): track 36.1 -> 35.1 mm
- net Net-(J2-Pin_8): track 35.4 -> 34.4 mm
- net Net-(J2-Pin_7): track 34.8 -> 33.8 mm
- net Net-(J2-Pin_6): track 35.4 -> 34.4 mm
- net Net-(J2-Pin_5): track 35.5 -> 34.5 mm
- net Net-(J2-Pin_4): track 36.2 -> 35.2 mm
- net Net-(J2-Pin_3): track 36.9 -> 35.9 mm
- net Net-(J2-Pin_2): track 37.6 -> 36.6 mm
- net Net-(J2-Pin_12): track 38.2 -> 37.2 mm
- net Net-(J2-Pin_11): track 37.5 -> 36.5 mm
- net Net-(J2-Pin_10): track 36.8 -> 35.8 mm
- net Net-(J2-Pin_1): track 38.2 -> 37.2 mm
Changed lines of the file:
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@@
 		(capping no)
 		(filling no)
-		(zone_defaults)
 		(pcbplotparams
 			(layerselection 0x00000000_00000000_55555555_5755f5ff)
@@
 			(outputformat 1)
 			(mirror no)
-			(drillshape 1)
+			(drillshape 0)
 			(scaleselection 1)
-			(outputdirectory "")
+			(outputdirectory "./")
 		)
 	)
 	(footprint "CONN12X1_2317507:CONN12X1_2317507-1_TEC"
 		(layer "F.Cu")
-		(at 201.5 104 180)
+		(at 201.5 103 180)
 		(tags "2317507-1 ")
 		(property "Reference" "J1"
@@
 	)
 	(segment
-		(start 206.45 94.4623)
+		(start 206.45 93.4623)
 		(end 206.45 92.05)
 		(width 0.25)
@@
 	(segment
 		(start 205.55 90.45)
-		(end 205.55 94.4623)
+		(end 205.55 93.4623)
 		(width 0.25)
 		(layer "F.Cu")
@@
 	(segment
 		(start 204.649999 88.350001)
-		(end 204.649999 94.4623)
+		(end 204.649999 93.4623)
 		(width 0.25)
 		(layer "F.Cu")
@@
 	(segment
 		(start 203.750001 86.249999)
-		(end 203.750001 94.4623)
+		(end 203.750001 93.4623)
 		(width 0.25)
 		(layer "F.Cu")
@@
 	(segment
 		(start 202.85 85.15)
-		(end 202.85 94.4623)
+		(end 202.85 93.4623)
 		(width 0.25)
 		(layer "F.Cu")
@@
 	(segment
 		(start 201.949999 60.930001)
-		(end 201.949999 94.4623)
+		(end 201.949999 93.4623)
 		(width 0.25)
 		(layer "F.Cu")
@@
 	(segment
 		(start 201.050001 60.710001)
-		(end 201.050001 94.4623)
+		(end 201.050001 93.4623)
 		(width 0.25)
 		(layer "F.Cu")
@@
 	(segment
 		(start 200.15 85.65)
-		(end 200.15 94.4623)
+		(end 200.15 93.4623)
 		(width 0.25)
 		(layer "F.Cu")
@@
 	(segment
 		(start 199.249999 87.249999)
-		(end 199.249999 94.4623)
+		(end 199.249999 93.4623)
 		(width 0.25)
 		(layer "F.Cu")
@@
 	(segment
 		(start 198.349999 88.849999)
-		(end 198.349999 94.4623)
+		(end 198.349999 93.4623)
 		(width 0.25)
 		(layer "F.Cu")
@@
 	(segment
 		(start 197.45 90.45)
-		(end 197.45 94.4623)
+		(end 197.45 93.4623)
 		(width 0.25)
 		(layer "F.Cu")
@@
 	(segment
 		(start 196.55 92.05)
-		(end 196.55 94.4623)
-		(width 0.25)
-		(layer "F.Cu")
+		(end 196.55 93.4623)
+		(width 0.25)
+		(layer "F.Cu")
